File: pneumatics/pneumatics.brd (EAGLE design)
At the start: 46.7 x 38.1 mm, 26 parts, among them U1 TPIC6A596

Commit message: Intermediate board
Parts:
- removed U$1: ATTINY84ATTINY84-20MU, SparkFun-IC-Microcontroller:QFN20
- added J3: AVR_SPI_PROG_3X2NS, SparkFun-Connectors:2X3-NS
- added U$2: ATTINY84, SparkFun-IC-Microcontroller:SO14
- moved C1 18.1 mm to (19.8, 15.0)
- moved C2 16.8 mm to (19.8, 17.3)
- moved SV1 11.5 mm to (8.89, 6.10)
- moved R1 8.89 mm to (20.3, 32.8)
- moved LED1 6.86 mm to (17.3, 32.8)
- moved 16 4.13 mm to (36.6, 14.7)
- moved 5 3.81 mm to (32.0, 14.7)
- moved 12V-TO-5V 3.53 mm to (13.5, 14.5), turned to 180 degrees
- moved 15 3.45 mm to (36.6, 19.6)
- moved 4 3.09 mm to (7.11, 14.7)
- moved 6 3.06 mm to (32.0, 19.6)
- moved 12 3.05 mm to (2.54, 14.7)
- moved 14 2.97 mm to (36.6, 24.4)
- moved R2 2.90 mm to (26.9, 17.3)
- moved 13 2.79 mm to (36.6, 29.2)
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Connections:
- removed net ENABLE: U$1.20, U1.9
- removed net SCL: SV1.2, U$1.1
- removed net SDA: SV1.1, U$1.16
- new net ENABLE/MISO: J3.1, U$2.8, U1.9
- new net RESET: J3.5, U$2.4
- new net SCL/SCK: J3.3, SV1.2, U$2.9
- new net SDA/MOSI: J3.4, SV1.1, U$2.7
- net +5V: now also J3.2, U$2.1; no longer U$1.9
- net GND: now also J3.6, U$2.14; no longer U$1.8
- net RCLK: now also U$2.12; no longer U$1.2
- net SERIAL_IN: now also U$2.13; no longer U$1.5
- net SRCLK: now also U$2.10; no longer U$1.4
- net SRCLR: now also U$2.11; no longer U$1.3
Routing:
- net +5V: track 0.00 -> 27.4 mm
- net SOL_3A: track 0.00 -> 14.3 mm
- net SOL_2B: track 0.00 -> 13.3 mm
- net SOL_3B: track 0.00 -> 11.2 mm
- net SOL_2A: track 0.00 -> 10.0 mm
- net SOL_4B: track 0.00 -> 9.35 mm
- net SOL_4A: track 0.00 -> 8.83 mm
- net SOL_1A: track 0.00 -> 8.34 mm
- net SOL_1B: track 0.00 -> 7.81 mm
- net N$1: track 0.00 -> 6.41 mm
- net N$7: track 0.00 -> 1.45 mm

Commit message: Done?
Parts:
- moved J3 3.10 mm to (23.9, 6.35)
- moved 5 3.06 mm to (32.3, 17.8)
- moved 6 3.06 mm to (32.3, 22.6)
- moved 8 3.06 mm to (32.3, 32.3)
- moved 1 3.06 mm to (7.37, 32.3)
- moved 11 3.06 mm to (2.79, 22.6)
- moved 12 3.06 mm to (2.79, 17.8)
- moved 13 3.06 mm to (36.8, 32.3)
- moved 15 3.06 mm to (36.8, 22.6)
- moved 16 3.06 mm to (36.8, 17.8)
- moved 3 3.06 mm to (7.37, 22.6)
- moved 4 3.06 mm to (7.37, 17.8)
- moved 9 3.06 mm to (2.79, 32.3)
- moved C2 3.06 mm to (20.1, 20.3)
- moved LED1 3.06 mm to (17.5, 35.8)
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Connections:
- net SCL/SCK: now also SV1.1; no longer SV1.2
- net SDA/MOSI: now also SV1.2; no longer SV1.1
Routing:
- net ENABLE/MISO: track 0.00 -> 37.5 mm, vias 0 -> 2
- net SERIAL_IN: track 0.00 -> 22.6 mm, vias 0 -> 2
- net SCL/SCK: track 0.00 -> 21.8 mm, vias 0 -> 3
- net SDA/MOSI: track 0.00 -> 21.3 mm, vias 0 -> 1
- net SRCLR: track 0.00 -> 15.4 mm, vias 0 -> 2
- net SRCLK: track 0.00 -> 13.0 mm
- net RCLK: track 0.00 -> 11.9 mm, vias 0 -> 2
- net +12V: track 0.00 -> 11.1 mm
- net RESET: track 0.00 -> 6.26 mm
- net +5V: track 27.4 -> 32.4 mm
- added copper zone on layer 1, net +12V
- added copper zone on layer 1, net GND
Other:
- board size 46.7 x 38.1 mm -> 39.8 x 38.1 mm
- board text added: "Pneumatics Board v1.0 Rov XX Jason King"
